Commit message: Adding prefix

File: description/urdf/diffbot_description.urdf.xacro (robot description, xacro)
@@ -13,13 +13,13 @@
         </material>
         <!-- BASE LINK -->
-        <link name="base_link">
+        <link name="${prefix}base_link">
         </link>
         <!-- CHASSIS LINK -->
-        <joint name="chassis_joint" type="fixed">
-            <parent link="base_link"/>
-            <child link="chassis"/>
+        <joint name="${prefix}chassis_joint" type="fixed">
+            <parent link="${prefix}base_link"/>
+            <child link="${prefix}chassis"/>
             <origin xyz="-0.07 0 0"/>
         </joint>
-        <link name="chassis">
+        <link name="${prefix}chassis">
             <visual>
                 <origin xyz="0.07 0 0.003"/>
@@ -40,5 +40,5 @@
             </xacro:inertial_cylinder>
         </link>
-        <gazebo reference="chassis">
+        <gazebo reference="${prefix}chassis">
             <material>
                 Gazebo/Red
@@ -46,11 +46,11 @@
         </gazebo>
         <!-- LEFT WHEEL LINK -->
-        <joint name="left_wheel_joint" type="continuous">
-            <parent link="base_link"/>
-            <child link="left_wheel"/>
+        <joint name="${prefix}left_wheel_joint" type="continuous">
+            <parent link="${prefix}base_link"/>
+            <child link="${prefix}left_wheel"/>
             <origin xyz="0 0.085 0" rpy="-${pi/2} 0 0" />
             <axis xyz="0 0 1"/>
         </joint>
-        <link name="left_wheel">
+        <link name="${prefix}left_wheel">
             <visual>
                 <geometry>
@@ -69,5 +69,5 @@
             </xacro:inertial_cylinder>
         </link>
-        <gazebo reference="left_wheel">
+        <gazebo reference="${prefix}left_wheel">
             <material>
                 Gazebo/Black
@@ -75,11 +75,11 @@
         </gazebo>
         <!-- RIGHT WHEEL LINK -->
-        <joint name="right_wheel_joint" type="continuous">
-            <parent link="base_link"/>
-            <child link="right_wheel"/>
+        <joint name="${prefix}right_wheel_joint" type="continuous">
+            <parent link="${prefix}base_link"/>
+            <child link="${prefix}right_wheel"/>
             <origin xyz="0 -0.085 0" rpy="${pi/2} 0 0"/>
             <axis xyz="0 0 -1"/>
         </joint>
-        <link name="right_wheel">
+        <link name="${prefix}right_wheel">
             <visual>
                 <geometry>
@@ -98,5 +98,5 @@
             </xacro:inertial_cylinder>
         </link>
-        <gazebo reference="right_wheel">
+        <gazebo reference="${prefix}right_wheel">
             <material>
                 Gazebo/Black
@@ -104,10 +104,10 @@
         </gazebo>
         <!-- CASTER WHEEL LINK -->
-        <joint name="caster_wheel_joint" type="fixed">
-            <parent link="chassis"/>
-            <child link="caster_wheel"/>
+        <joint name="${prefix}caster_wheel_joint" type="fixed">
+            <parent link="${prefix}chassis"/>
+            <child link="${prefix}caster_wheel"/>
             <origin xyz="0.005 0 -0.022"/>
         </joint>
-        <link name="caster_wheel">
+        <link name="${prefix}caster_wheel">
             <visual>
                 <geometry>
@@ -126,5 +126,5 @@
             </xacro:inertial_sphere>
         </link>
-        <gazebo reference="caster_wheel">
+        <gazebo reference="${prefix}caster_wheel">
             <material>
                 Gazebo/White
