Commit message: URDF Updated for TI-RSLK Max

File: description/ros2_control/diffbot.ros2_control.xacro (robot description, xacro)
@@ -7,7 +7,7 @@
         <param name="left_wheel_name">left_wheel_joint</param>
         <param name="right_wheel_name">right_wheel_joint</param>
-        <param name="loop_rate">30</param>
-        <param name="device">/dev/serial/by-path/platform-fd500000.pcie-pci-0000:01:00.0-usb-0:1.3:1.0-port0</param>
-        <param name="baud_rate">57600</param>
+        <param name="loop_rate">50</param>
+        <param name="device">/dev/ttyACM0</param>
+        <param name="baud_rate">9600</param>
         <param name="timeout_ms">1000</param>
         <param name="enc_counts_per_rev">3436</param>

File: description/urdf/diffbot.materials.xacro (robot description, xacro)
@@ -24,5 +24,5 @@
   </material>
   <material name="red">
-    <color rgba="0.8 0.0 0.0 1.0"/>
+    <color rgba="1.0 0.0 0.0 1.0"/>
   </material>
   <material name="white">

File: description/urdf/diffbot.urdf.xacro (robot description, xacro)
@@ -4,6 +4,4 @@
   <xacro:arg name="prefix" default="" />
   <xacro:include filename="$(find diffdrive_msp432)/urdf/diffbot_description.urdf.xacro" />
-  <!-- Import Rviz colors -->
-  <xacro:include filename="$(find diffdrive_msp432)/urdf/diffbot.materials.xacro" />
   <!-- Import diffbot ros2_control description -->
   <xacro:include filename="$(find diffdrive_msp432)/ros2_control/diffbot.ros2_control.xacro" />

File: description/urdf/diffbot_description.urdf.xacro (robot description, xacro)
@@ -1,161 +1,136 @@
 <?xml version="1.0"?>
 <robot xmlns:xacro="http://www.ros.org/wiki/xacro">
-  <xacro:macro name="diffbot" params="prefix">
-  <!-- Constants for robot dimensions -->
-  <xacro:property name="PI" value="3.1415926535897931"/>
-  <xacro:property name="base_mass" value="0.3" /> <!-- arbitrary value for base mass -->
-  <xacro:property name="base_width" value="0.1" />
-  <xacro:property name="base_length" value="0.1" />
-  <xacro:property name="base_height" value="0.05" />
-  <xacro:property name="wheel_mass" value="0.3" /> <!-- arbitrary value for wheel mass -->
-  <xacro:property name="wheel_len" value="0.020" />
-  <xacro:property name="wheel_radius" value="0.015" />
-  <xacro:property name="caster_wheel_mass" value="0.1" /> <!-- arbitrary value for caster wheel mass -->
-  <xacro:property name="caster_wheel_radius" value="0.015" />
-  <xacro:property name="z_offset" value="-${base_height/2}" /> <!-- Space btw top of beam and the each joint -->
-  <!-- Base Link -->
-  <link name="${prefix}base_link">
-    <collision>
-      <origin xyz="0 0 0" rpy="0 0 0"/>
-      <geometry>
-        <box size="${base_width} ${base_length} ${base_height}"/>
-      </geometry>
-    </collision>
-    <visual>
-      <origin xyz="0 0 ${base_height/2}" rpy="0 0 0"/>
-      <geometry>
-        <box size="${base_width} ${base_length} ${base_height}"/>
-      </geometry>
-      <material name="orange"/>
-    </visual>
-    <inertial>
-      <origin xyz="0 0 0" rpy="0 0 0"/>
-      <mass value="${base_mass}"/>
-      <inertia
-        ixx="${base_mass / 12.0 * (base_length*base_length + base_height*base_height)}" ixy="0.0" ixz="0.0"
-        iyy="${base_mass / 12.0 * (base_height*base_height + base_width*base_width)}" iyz="0.0"
-        izz="${base_mass / 12.0 * (base_width*base_width + base_length*base_length)}"/>
-      </inertial>
-    </link>
-    <joint name="${prefix}left_wheel_joint" type="continuous">
-      <parent link="${prefix}base_link"/>
-      <child link="${prefix}left_wheel"/>
-      <origin xyz="0 -${base_width/2} ${z_offset}" rpy="0 0 0"/>
-      <axis xyz="0 1 0"/>
-      <dynamics damping="0.2"/>
-    </joint>
-    <!-- left wheel Link -->
-    <link name="${prefix}left_wheel">
-      <collision>
-        <origin xyz="0 0 0" rpy="${PI/2} 0 0"/>
-        <geometry>
-          <cylinder length="${wheel_len}" radius="${wheel_radius}"/>
-        </geometry>
-      </collision>
-      <visual>
-        <origin xyz="0 0 0" rpy="${PI/2} 0 0"/>
-        <geometry>
-          <cylinder length="${wheel_len}" radius="${wheel_radius}"/>
-        </geometry>
-        <material name="black"/>
-      </visual>
-      <inertial>
-        <origin xyz="0 0 0" rpy="${PI/2} 0 0"/>
-        <mass value="${wheel_mass}"/>
-        <inertia
-          ixx="${wheel_mass / 12.0 * (3*wheel_radius + wheel_len*wheel_len)}" ixy="0.0" ixz="0.0"
-          iyy="${wheel_mass / 12.0 * wheel_radius*wheel_radius}" iyz="0.0"
-          izz="${wheel_mass / 12.0 * wheel_radius*wheel_radius}"/>
-        </inertial>
-      </link>
-    <joint name="${prefix}right_wheel_joint" type="continuous">
-      <parent link="${prefix}base_link"/>
-      <child link="${prefix}right_wheel"/>
-      <origin xyz="0 ${base_width/2} ${z_offset}" rpy="0 0 0"/>
-      <axis xyz="0 1 0"/>
-      <dynamics damping="0.2"/>
-    </joint>
-    <!-- right wheel Link -->
-    <link name="${prefix}right_wheel">
-      <collision>
-        <origin xyz="0 0 0" rpy="${PI/2} 0 0"/>
-        <geometry>
-          <cylinder length="${wheel_len}" radius="${wheel_radius}"/>
-        </geometry>
-      </collision>
-      <visual>
-        <origin xyz="0 0 0" rpy="${PI/2} 0 0"/>
-        <geometry>
-          <cylinder length="${wheel_len}" radius="${wheel_radius}"/>
-        </geometry>
-        <material name="black"/>
-      </visual>
-      <inertial>
-        <origin xyz="0 0 0" rpy="${PI/2} 0 0"/>
-        <mass value="${wheel_mass}"/>
-        <inertia
-          ixx="${wheel_mass / 12.0 * (3*wheel_radius + wheel_len*wheel_len)}" ixy="0.0" ixz="0.0"
-          iyy="${wheel_mass / 12.0 * wheel_radius*wheel_radius}" iyz="0.0"
-          izz="${wheel_mass / 12.0 * wheel_radius*wheel_radius}"/>
-        </inertial>
-      </link>
-    <joint name="${prefix}caster_frontal_wheel_joint" type="fixed">
-      <parent link="${prefix}base_link"/>
-      <child link="${prefix}caster_frontal_wheel"/>
-      <origin xyz="${base_width/2 - caster_wheel_radius} 0 ${z_offset}" rpy="0 0 0"/>
-    </joint>
-    <!-- caster frontal wheel Link -->
-    <link name="${prefix}caster_frontal_wheel">
-      <collision>
-        <origin xyz="0 0 0" rpy="0 0 0"/>
-        <geometry>
-          <sphere radius="${caster_wheel_radius}"/>
-        </geometry>
-      </collision>
-      <visual>
-        <origin xyz="0 0 0" rpy="0 0 0"/>
-        <geometry>
-          <sphere radius="${caster_wheel_radius}"/>
-        </geometry>
-        <material name="white"/>
-      </visual>
-      <inertial>
-        <origin xyz="0 0 0" rpy="0 0 0"/>
-        <mass value="${caster_wheel_mass}"/>
-        <inertia
-          ixx="${caster_wheel_mass * 0.4 * (caster_wheel_radius * caster_wheel_radius)}" ixy="0.0" ixz="0.0"
-          iyy="${caster_wheel_mass * 0.4 * (caster_wheel_radius * caster_wheel_radius)}" iyz="0.0"
-          izz="${caster_wheel_mass * 0.4 * (caster_wheel_radius * caster_wheel_radius)}"/>
-        </inertial>
-      </link>
-    <joint name="${prefix}caster_rear_wheel_joint" type="fixed">
-      <parent link="${prefix}base_link"/>
-      <child link="${prefix}caster_rear_wheel"/>
-      <origin xyz="${-base_width/2 + caster_wheel_radius} 0 ${z_offset}" rpy="0 0 0"/>
-    </joint>
-    <!-- caster rear wheel Link -->
-    <link name="${prefix}caster_rear_wheel">
-      <collision>
-        <origin xyz="0 0 0" rpy="0 0 0"/>
-        <geometry>
-          <sphere radius="${caster_wheel_radius}"/>
-        </geometry>
-      </collision>
-      <visual>
-        <origin xyz="0 0 0" rpy="0 0 0"/>
-        <geometry>
-          <sphere radius="${caster_wheel_radius}"/>
-        </geometry>
-        <material name="white"/>
-      </visual>
-      <inertial>
-        <origin xyz="0 0 0" rpy="0 0 0"/>
-        <mass value="${caster_wheel_mass}"/>
-        <inertia
-          ixx="${caster_wheel_mass * 0.4 * (caster_wheel_radius * caster_wheel_radius)}" ixy="0.0" ixz="0.0"
-          iyy="${caster_wheel_mass * 0.4 * (caster_wheel_radius * caster_wheel_radius)}" iyz="0.0"
-          izz="${caster_wheel_mass * 0.4 * (caster_wheel_radius * caster_wheel_radius)}"/>
-        </inertial>
-      </link>
-  </xacro:macro>
+    <xacro:include filename="inertial_macros.xacro"/>
+    <xacro:macro name="diffbot" params="prefix">
+        <material name="white">
+            <color rgba="1 1 1 1"/>
+        </material>
+        <material name="red">
+            <color rgba="1 0 0 1"/>
+        </material>
+        <material name="black">
+            <color rgba="0 0 0 1"/>
+        </material>
+        <!-- BASE LINK -->
+        <link name="base_link">
+        </link>
+        <!-- CHASSIS LINK -->
+        <joint name="chassis_joint" type="fixed">
+            <parent link="base_link"/>
+            <child link="chassis"/>
+            <origin xyz="-0.07 0 0"/>
+        </joint>
+        <link name="chassis">
+            <visual>
+                <origin xyz="0.07 0 0.003"/>
+                <geometry>
+                    <cylinder radius="0.08" length="0.05"/>
+                </geometry>
+                <material name="red"/>
+            </visual>
+            <collision>
+                <origin xyz="0.07 0 0.003"/>
+                <geometry>
+                    <cylinder radius="0.08" length="0.05"/>
+                </geometry>
+                <material name="red"/>
+            </collision>
+            <xacro:inertial_cylinder mass="0.243" length="0.05" radius="0.08">
+                <origin xyz="0.07 0 0.003" rpy="0 0 0"/>
+            </xacro:inertial_cylinder>
+        </link>
+        <gazebo reference="chassis">
+            <material>
+                Gazebo/Red
+            </material>
+        </gazebo>
+        <!-- LEFT WHEEL LINK -->
+        <joint name="left_wheel_joint" type="continuous">
+            <parent link="base_link"/>
+            <child link="left_wheel"/>
+            <origin xyz="0 0.085 0" rpy="-${pi/2} 0 0" />
+            <axis xyz="0 0 1"/>
+        </joint>
+        <link name="left_wheel">
+            <visual>
+                <geometry>
+                    <cylinder radius="0.035" length="0.008"/>
+                </geometry>
+                <material name="black"/>
+            </visual>
+            <collision>
+                <geometry>
+                    <cylinder radius="0.035" length="0.008"/>
+                </geometry>
+                <material name="black"/>
+            </collision>
+            <xacro:inertial_cylinder mass="0.007" length="0.008" radius="0.035">
+                <origin xyz="0 0 0" rpy="0 0 0"/>
+            </xacro:inertial_cylinder>
+        </link>
+        <gazebo reference="left_wheel">
+            <material>
+                Gazebo/Black
+            </material>
+        </gazebo>
+        <!-- RIGHT WHEEL LINK -->
+        <joint name="right_wheel_joint" type="continuous">
+            <parent link="base_link"/>
+            <child link="right_wheel"/>
+            <origin xyz="0 -0.085 0" rpy="${pi/2} 0 0"/>
+            <axis xyz="0 0 -1"/>
+        </joint>
+        <link name="right_wheel">
+            <visual>
+                <geometry>
+                    <cylinder radius="0.035" length="0.008"/>
+                </geometry>
+                <material name="black"/>
+            </visual>
+            <collision>
+                <geometry>
+                    <cylinder radius="0.035" length="0.008"/>
+                </geometry>
+                <material name="black"/>
+            </collision>
+            <xacro:inertial_cylinder mass="0.007" length="0.008" radius="0.035">
+                <origin xyz="0 0 0" rpy="0 0 0"/>
+            </xacro:inertial_cylinder>
+        </link>
+        <gazebo reference="right_wheel">
+            <material>
+                Gazebo/Black
+            </material>
+        </gazebo>
+        <!-- CASTER WHEEL LINK -->
+        <joint name="caster_wheel_joint" type="fixed">
+            <parent link="chassis"/>
+            <child link="caster_wheel"/>
+            <origin xyz="0.005 0 -0.022"/>
+        </joint>
+        <link name="caster_wheel">
+            <visual>
+                <geometry>
+                    <sphere radius="0.0127"/>
+                </geometry>
+                <material name="white"/>
+            </visual>
+            <collision>
+                <geometry>
+                    <sphere radius="0.0127"/>
+                </geometry>
+                <material name="white"/>
+            </collision>
+            <xacro:inertial_sphere mass="0.0165" radius="0.0127">
+                <origin xyz="0 0 0" rpy="0 0 0"/>
+            </xacro:inertial_sphere>
+        </link>
+        <gazebo reference="caster_wheel">
+            <material>
+                Gazebo/White
+            </material>
+            <mu1 value="0.001"/>
+            <mu2 value="0.001"/>
+        </gazebo>
+    </xacro:macro>
 </robot>

Commit message: Multi-agent implementation fixed

File: description/ros2_control/diffbot.ros2_control.xacro (robot description, xacro)
@@ -17,10 +17,10 @@
         <param name="pid_o">50</param>
       </hardware>
-      <joint name="${prefix}left_wheel_joint">
+      <joint name="left_wheel_joint">
         <command_interface name="velocity"/>
         <state_interface name="position"/>
         <state_interface name="velocity"/>
       </joint>
-      <joint name="${prefix}right_wheel_joint">
+      <joint name="right_wheel_joint">
         <command_interface name="velocity"/>
         <state_interface name="position"/>

Commit message: Restoring branch Multi-agent

File: description/ros2_control/diffbot.ros2_control.xacro (robot description, xacro)
@@ -5,6 +5,6 @@
       <hardware>
         <plugin>diffdrive_msp432/DiffDriveMSP432Hardware</plugin>
-        <param name="left_wheel_name">${prefix}left_wheel_joint</param>
-        <param name="right_wheel_name">${prefix}right_wheel_joint</param>
+        <param name="left_wheel_name">left_wheel_joint</param>
+        <param name="right_wheel_name">right_wheel_joint</param>
         <param name="loop_rate">30</param>
         <param name="device">/dev/ttyACM0</param>

File: description/urdf/diffbot_description.urdf.xacro (robot description, xacro)
@@ -13,13 +13,13 @@
         </material>
         <!-- BASE LINK -->
-        <link name="${prefix}base_link">
+        <link name="base_link">
         </link>
         <!-- CHASSIS LINK -->
-        <joint name="${prefix}chassis_joint" type="fixed">
-            <parent link="${prefix}base_link"/>
-            <child link="${prefix}chassis"/>
+        <joint name="chassis_joint" type="fixed">
+            <parent link="base_link"/>
+            <child link="chassis"/>
             <origin xyz="-0.07 0 0"/>
         </joint>
-        <link name="${prefix}chassis">
+        <link name="chassis">
             <visual>
                 <origin xyz="0.07 0 0.003"/>
@@ -40,5 +40,5 @@
             </xacro:inertial_cylinder>
         </link>
-        <gazebo reference="${prefix}chassis">
+        <gazebo reference="chassis">
             <material>
                 Gazebo/Red
@@ -46,11 +46,11 @@
         </gazebo>
         <!-- LEFT WHEEL LINK -->
-        <joint name="${prefix}left_wheel_joint" type="continuous">
-            <parent link="${prefix}base_link"/>
-            <child link="${prefix}left_wheel"/>
+        <joint name="left_wheel_joint" type="continuous">
+            <parent link="base_link"/>
+            <child link="left_wheel"/>
             <origin xyz="0 0.085 0" rpy="-${pi/2} 0 0" />
             <axis xyz="0 0 1"/>
         </joint>
-        <link name="${prefix}left_wheel">
+        <link name="left_wheel">
             <visual>
                 <geometry>
@@ -69,5 +69,5 @@
             </xacro:inertial_cylinder>
         </link>
-        <gazebo reference="${prefix}left_wheel">
+        <gazebo reference="left_wheel">
             <material>
                 Gazebo/Black
@@ -75,11 +75,11 @@
         </gazebo>
         <!-- RIGHT WHEEL LINK -->
-        <joint name="${prefix}right_wheel_joint" type="continuous">
-            <parent link="${prefix}base_link"/>
-            <child link="${prefix}right_wheel"/>
+        <joint name="right_wheel_joint" type="continuous">
+            <parent link="base_link"/>
+            <child link="right_wheel"/>
             <origin xyz="0 -0.085 0" rpy="${pi/2} 0 0"/>
             <axis xyz="0 0 -1"/>
         </joint>
-        <link name="${prefix}right_wheel">
+        <link name="right_wheel">
             <visual>
                 <geometry>
@@ -98,5 +98,5 @@
             </xacro:inertial_cylinder>
         </link>
-        <gazebo reference="${prefix}right_wheel">
+        <gazebo reference="right_wheel">
             <material>
                 Gazebo/Black
@@ -104,10 +104,10 @@
         </gazebo>
         <!-- CASTER WHEEL LINK -->
-        <joint name="${prefix}caster_wheel_joint" type="fixed">
-            <parent link="${prefix}chassis"/>
-            <child link="${prefix}caster_wheel"/>
+        <joint name="caster_wheel_joint" type="fixed">
+            <parent link="chassis"/>
+            <child link="caster_wheel"/>
             <origin xyz="0.005 0 -0.022"/>
         </joint>
-        <link name="${prefix}caster_wheel">
+        <link name="caster_wheel">
             <visual>
                 <geometry>
@@ -126,5 +126,5 @@
             </xacro:inertial_sphere>
         </link>
-        <gazebo reference="${prefix}caster_wheel">
+        <gazebo reference="caster_wheel">
             <material>
                 Gazebo/White

Commit message: Implementation mejoras + simulador

File: description/ros2_control/diffbot.ros2_control.xacro (robot description, xacro)
@@ -1,8 +1,13 @@
 <?xml version="1.0"?>
 <robot xmlns:xacro="http://www.ros.org/wiki/xacro">
-  <xacro:macro name="diffbot_ros2_control" params="name prefix">
+  <xacro:macro name="diffbot_ros2_control" params="name prefix use_sim">
     <ros2_control name="${name}" type="system">
       <hardware>
-        <plugin>diffdrive_msp432/DiffDriveMSP432Hardware</plugin>
+        <xacro:if value="${use_sim}">
+          <plugin>diffdrive_msp432/DiffDriveMSP432SimHardware</plugin>
+        </xacro:if>
+        <xacro:unless value="${use_sim}">
+          <plugin>diffdrive_msp432/DiffDriveMSP432Hardware</plugin>
+        </xacro:unless>
         <param name="left_wheel_name">left_wheel_joint</param>
         <param name="right_wheel_name">right_wheel_joint</param>

File: description/urdf/diffbot.urdf.xacro (robot description, xacro)
@@ -3,4 +3,5 @@
 <robot xmlns:xacro="http://www.ros.org/wiki/xacro" name="diffdrive_robot">
   <xacro:arg name="prefix" default="" />
+  <xacro:arg name="use_sim" default="false" />
   <xacro:include filename="$(find diffdrive_msp432)/urdf/diffbot_description.urdf.xacro" />
   <!-- Import diffbot ros2_control description -->
@@ -8,4 +9,4 @@
   <xacro:diffbot prefix="$(arg prefix)" />
   <xacro:diffbot_ros2_control
-    name="DiffBot" prefix="$(arg prefix)" />
+    name="DiffBot" prefix="$(arg prefix)" use_sim="$(arg use_sim)" />
 </robot>
